Commit message: Fix mimic joints for Gazebo compatibility

File: robotiq_description/urdf/robotiq_2f_85_macro.urdf.xacro (robot description, xacro)
@@ -245,5 +245,5 @@
             <origin xyz="-0.03060114 0.0 0.05490452" rpy="0 0 0" />
             <limit lower="-0.8" upper="0.0" velocity="0.5" effort="50" />
-            <mimic joint="${prefix}robotiq_85_left_knuckle_joint" multiplier="-1" />
+            <dynamics damping ="0.5" friction="0.1"/>
         </joint>
         <joint name="${prefix}robotiq_85_left_finger_joint" type="fixed">
@@ -262,5 +262,5 @@
             <axis xyz="0 -1 0" />
             <origin xyz="0.0127 0.0 0.06142" rpy="0 0 0" />
-            <mimic joint="${prefix}robotiq_85_left_knuckle_joint" />
+            <dynamics damping="0.5" friction="0.1"/>
             <limit lower="0.0" upper="0.8" velocity="0.5" effort="50" />
         </joint>
@@ -270,5 +270,5 @@
             <axis xyz="0 -1 0" />
             <origin xyz="-0.0127 0.0 0.06142" rpy="0 0 0" />
-            <mimic joint="${prefix}robotiq_85_left_knuckle_joint" multiplier="-1" />
+            <dynamics damping="0.5" friction="0.1" />
             <limit lower="-0.8" upper="0.0" velocity="0.5" effort="50" />
         </joint>
@@ -278,5 +278,5 @@
             <axis xyz="0 -1 0" />
             <origin xyz="0.00563134 0.0 0.04718515" rpy="0 0 0" />
-            <mimic joint="${prefix}robotiq_85_left_knuckle_joint" multiplier="-1" />
+            <dynamic damping="0.5" friction="0.1" />
             <limit lower="-0.8" upper="0.0" velocity="0.5" effort="50" />
         </joint>
@@ -286,5 +286,5 @@
             <axis xyz="0 -1 0" />
             <origin xyz="-0.00563134 0.0 0.04718515" rpy="0 0 0" />
-            <mimic joint="${prefix}robotiq_85_left_knuckle_joint" />
+            <dynamics damping="0.5" friction="0.1" />
             <limit lower="0.0" upper="0.8" velocity="0.5" effort="50" />
         </joint>
