Commit message: feat: redesign gripper to 3-fingered variant with updated ros2_control and controllers

File: robotiq_description/urdf/2f_85.ros2_control.xacro (robot description, xacro)
@@ -17,7 +17,5 @@
         gripper_closed_position:=0.7929">
         <ros2_control name="${name}" type="system">
-            <!-- Plugins -->
             <hardware>
-                <!-- Set use_dummy to true to connect to a dummy driver for testing purposes. -->
                 <param name="use_dummy">false</param>
                 <xacro:if value="${sim_isaac}">
@@ -45,7 +43,5 @@
                 </xacro:unless>
             </hardware>
-            <!-- Joint interfaces -->
-            <!-- With Gazebo or Hardware, they handle mimic joints, so we only need this command interface activated -->
-            <joint name="${prefix}robotiq_85_left_knuckle_joint">
+            <joint name="${prefix}robotiq_85_finger_1_knuckle_joint">
                 <command_interface name="position" />
                 <state_interface name="position">
@@ -54,7 +50,20 @@
                 <state_interface name="velocity"/>
             </joint>
-            <!-- When simulating we need to include the rest of the gripper joints -->
+            <joint name="${prefix}robotiq_85_finger_2_knuckle_joint">
+                <command_interface name="position" />
+                <state_interface name="position">
+                    <param name="initial_value">${gripper_closed_position}</param>
+                </state_interface>
+                <state_interface name="velocity"/>
+            </joint>
+            <joint name="${prefix}robotiq_85_finger_3_knuckle_joint">
+                <command_interface name="position" />
+                <state_interface name="position">
+                    <param name="initial_value">${gripper_closed_position}</param>
+                </state_interface>
+                <state_interface name="velocity"/>
+            </joint>
             <xacro:if value="${use_fake_hardware or sim_isaac or sim_gazebo}">
-                <joint name="${prefix}robotiq_85_right_knuckle_joint">
+                <joint name="${prefix}robotiq_85_finger_1_inner_knuckle_joint">
                     <xacro:unless value="${sim_gazebo}">
                         <state_interface name="position"/>
@@ -62,5 +71,5 @@
                     </xacro:unless>
                 </joint>
-                <joint name="${prefix}robotiq_85_left_inner_knuckle_joint">
+                <joint name="${prefix}robotiq_85_finger_1_finger_tip_joint">
                     <xacro:unless value="${sim_gazebo}">
                         <state_interface name="position"/>
@@ -68,5 +77,5 @@
                     </xacro:unless>
                 </joint>
-                <joint name="${prefix}robotiq_85_right_inner_knuckle_joint">
+                <joint name="${prefix}robotiq_85_finger_2_inner_knuckle_joint">
                     <xacro:unless value="${sim_gazebo}">
                         <state_interface name="position"/>
@@ -74,5 +83,5 @@
                     </xacro:unless>
                 </joint>
-                <joint name="${prefix}robotiq_85_left_finger_tip_joint">
+                <joint name="${prefix}robotiq_85_finger_2_finger_tip_joint">
                     <xacro:unless value="${sim_gazebo}">
                         <state_interface name="position"/>
@@ -80,5 +89,11 @@
                     </xacro:unless>
                 </joint>
-                <joint name="${prefix}robotiq_85_right_finger_tip_joint">
+                <joint name="${prefix}robotiq_85_finger_3_inner_knuckle_joint">
+                    <xacro:unless value="${sim_gazebo}">
+                        <state_interface name="position"/>
+                        <state_interface name="velocity"/>
+                    </xacro:unless>
+                </joint>
+                <joint name="${prefix}robotiq_85_finger_3_finger_tip_joint">
                     <xacro:unless value="${sim_gazebo}">
                         <state_interface name="position"/>
@@ -87,5 +102,4 @@
                 </joint>
             </xacro:if>
-            <!-- Only add this with fake hardware mode -->
             <xacro:unless value="${sim_gazebo or sim_isaac}">
                 <gpio name="reactivate_gripper">

File: robotiq_description/urdf/robotiq_2f_85_macro.urdf.xacro (robot description, xacro)
@@ -19,7 +19,5 @@
         gripper_max_force:=235.0
         gripper_closed_position:=0.7929">
-        <!-- ros2 control include -->
         <xacro:include filename="$(find robotiq_description)/urdf/2f_85.ros2_control.xacro" />
-        <!-- if we are simulating or directly communicating with the gripper we need a ros2 control instance -->
         <xacro:if value="${include_ros2_control}">
             <xacro:robotiq_gripper_ros2_control
@@ -55,176 +53,4 @@
             </inertial>
         </link>
-        <link name="${prefix}robotiq_85_left_knuckle_link">
-            <visual>
-                <geometry>
-                    <mesh filename="package://robotiq_description/meshes/visual/2f_85/left_knuckle.dae" />
-                </geometry>
-            </visual>
-            <collision>
-                <geometry>
-                    <mesh filename="package://robotiq_description/meshes/collision/2f_85/left_knuckle.stl" />
-                </geometry>
-            </collision>
-            <inertial>
-                <origin xyz="0.01213197 0.0002 -0.00058647" rpy="0 0 0" />
-                <mass value="1.384773208e-02" />
-                <inertia ixx="3.5232e-7" iyy="2.31944e-6" izz="2.23136e-6" ixy="0.0" ixz="1.1744e-7" iyz="0" />
-            </inertial>
-        </link>
-        <link name="${prefix}robotiq_85_right_knuckle_link">
-            <visual>
-                <geometry>
-                    <mesh filename="package://robotiq_description/meshes/visual/2f_85/right_knuckle.dae" />
-                </geometry>
-            </visual>
-            <collision>
-                <geometry>
-                    <mesh filename="package://robotiq_description/meshes/collision/2f_85/right_knuckle.stl" />
-                </geometry>
-            </collision>
-            <inertial>
-                <origin xyz="-0.01213197 0.0002 -0.00058647" rpy="0 0 0" />
-                <mass value="1.384773208e-02" />
-                <inertia ixx="3.5232e-7" iyy="2.31944e-6" izz="2.23136e-6" ixy="0.0" ixz="-1.1744e-7" iyz="0.0" />
-            </inertial>
-        </link>
-        <link name="${prefix}robotiq_85_left_finger_link">
-            <visual>
-                <geometry>
-                    <mesh filename="package://robotiq_description/meshes/visual/2f_85/left_finger.dae" />
-                </geometry>
-            </visual>
-            <collision>
-                <geometry>
-                    <mesh filename="package://robotiq_description/meshes/collision/2f_85/left_finger.stl" />
-                </geometry>
-            </collision>
-            <inertial>
-                <origin xyz="0.00346899 -0.00079447 0.01867121" rpy="0 0 0" />
-                <mass value="4.260376752e-02" />
-                <inertia ixx="1.385792000000000e-05" iyy="1.183208e-05" izz="5.19672e-06" ixy="0.0" ixz="-2.17264e-06" iyz="0.0" />
-            </inertial>
-        </link>
-        <link name="${prefix}robotiq_85_right_finger_link">
-            <visual>
-                <geometry>
-                    <mesh filename="package://robotiq_description/meshes/visual/2f_85/right_finger.dae" />
-                </geometry>
-            </visual>
-            <collision>
-                <geometry>
-                    <mesh filename="package://robotiq_description/meshes/collision/2f_85/right_finger.stl" />
-                </geometry>
-            </collision>
-            <inertial>
-                <origin xyz="-0.00346899 -5.53e-06 0.01867121" rpy="0 0 0" />
-                <mass value="4.260376752000000e-02" />
-                <inertia ixx="1.385792e-05" iyy="1.183208e-05" izz="5.19672e-06" ixy="0.0" ixz="2.17264e-06" iyz="0.0" />
-            </inertial>
-        </link>
-        <link name="${prefix}robotiq_85_left_inner_knuckle_link">
-            <visual>
-                <geometry>
-                    <mesh filename="package://robotiq_description/meshes/visual/2f_85/left_inner_knuckle.dae" />
-                </geometry>
-            </visual>
-            <collision>
-                <geometry>
-                    <mesh filename="package://robotiq_description/meshes/collision/2f_85/left_inner_knuckle.stl" />
-                </geometry>
-            </collision>
-            <inertial>
-                <origin xyz="0.01897699 0.00015001 0.02247101" rpy="0 0 0" />
-                <mass value="2.969376448e-02" />
-                <inertia ixx="9.57136e-06" iyy="8.69056e-06" izz="8.19144e-06" ixy="0.0" ixz="-3.93424e-06" iyz="0.0" />
-            </inertial>
-        </link>
-        <link name="${prefix}robotiq_85_right_inner_knuckle_link">
-            <visual>
-                <geometry>
-                    <mesh filename="package://robotiq_description/meshes/visual/2f_85/right_inner_knuckle.dae" />
-                </geometry>
-            </visual>
-            <collision>
-                <geometry>
-                    <mesh filename="package://robotiq_description/meshes/collision/2f_85/right_inner_knuckle.stl" />
-                </geometry>
-            </collision>
-            <inertial>
-                <origin xyz="-0.01926824 5.001e-05 0.02222178" rpy="0 0 0" />
-                <mass value="2.969376448e-02" />
-                <inertia ixx="9.42456e-06" iyy="8.69056e-06" izz="8.33824e-06" ixy="0.0" ixz="3.9636e-06" iyz="0.0" />
-            </inertial>
-        </link>
-        <link name="${prefix}robotiq_85_left_finger_tip_link">
-            <visual>
-                <geometry>
-                    <mesh filename="package://robotiq_description/meshes/visual/2f_85/left_finger_tip.dae" />
-                </geometry>
-            </visual>
-            <collision>
-                <geometry>
-                    <mesh filename="package://robotiq_description/meshes/collision/2f_85/left_finger_tip.stl" />
-                </geometry>
-                <surface>
-                    <friction>
-                    <ode>
-                        <mu1>100000.0</mu1>
-                        <mu2>100000.0</mu2>
-                    </ode>
-                    </friction>
-                    <contact>
-                    <ode>
-                        <kp>1e+5</kp>
-                        <kd>1</kd>
-                        <soft_cfm>0</soft_cfm>
-                        <soft_erp>0.2</soft_erp>
-                        <minDepth>0.002</minDepth>
-                        <maxVel>0</maxVel>
-                    </ode>
-                    </contact>
-                </surface>
-            </collision>
-            <inertial>
-                <origin xyz="-0.01456706 -0.0008 0.01649701" rpy="0 0 0" />
-                <mass value="4.268588744e-02" />
-                <inertia ixx="1.048152e-05" iyy="1.197888e-05" izz="4.22784e-06" ixy="0.0" ixz="3.5232e-6" iyz="0.0" />
-            </inertial>
-        </link>
-        <link name="${prefix}robotiq_85_right_finger_tip_link">
-            <visual>
-                <geometry>
-                    <mesh filename="package://robotiq_description/meshes/visual/2f_85/right_finger_tip.dae" />
-                </geometry>
-            </visual>
-            <collision>
-                <geometry>
-                    <mesh filename="package://robotiq_description/meshes/collision/2f_85/right_finger_tip.stl" />
-                </geometry>
-                <surface>
-                    <friction>
-                    <ode>
-                        <mu1>100000.0</mu1>
-                        <mu2>100000.0</mu2>
-                    </ode>
-                    </friction>
-                    <contact>
-                    <ode>
-                        <kp>1e+5</kp>
-                        <kd>1</kd>
-                        <soft_cfm>0</soft_cfm>
-                        <soft_erp>0.2</soft_erp>
-                        <minDepth>0.002</minDepth>
-                        <maxVel>0</maxVel>
-                    </ode>
-                    </contact>
-                </surface>
-            </collision>
-            <inertial>
-                <origin xyz="0.01456706 5e-05 0.01649701" rpy="0 0 0" />
-                <mass value="4.268588744e-02" />
-                <inertia ixx="1.048152e-05" iyy="1.197888e-05" izz="4.22784e-06" ixy="0.0" ixz="-3.5232e-06" iyz="0.0" />
-            </inertial>
-        </link>
         <joint name="${prefix}robotiq_85_base_joint" type="fixed">
             <parent link="${parent}" />
@@ -232,61 +58,123 @@
             <xacro:insert_block name="origin" />
         </joint>
-        <joint name="${prefix}robotiq_85_left_knuckle_joint" type="revolute">
-            <parent link="${prefix}robotiq_85_base_link" />
-            <child link="${prefix}robotiq_85_left_knuckle_link" />
-            <axis xyz="0 -1 0" />
-            <origin xyz="0.03060114 0.0 0.05490452" rpy="0 0 0" />
-            <limit lower="0.0" upper="0.8" velocity="0.5" effort="50" />
-        </joint>
-        <joint name="${prefix}robotiq_85_right_knuckle_joint" type="revolute">
-            <parent link="${prefix}robotiq_85_base_link" />
-            <child link="${prefix}robotiq_85_right_knuckle_link" />
-            <axis xyz="0 -1 0" />
-            <origin xyz="-0.03060114 0.0 0.05490452" rpy="0 0 0" />
-            <limit lower="-0.8" upper="0.0" velocity="0.5" effort="50" />
-            <dynamics damping ="0.5" friction="0.1"/>
-        </joint>
-        <joint name="${prefix}robotiq_85_left_finger_joint" type="fixed">
-            <parent link="${prefix}robotiq_85_left_knuckle_link" />
-            <child link="${prefix}robotiq_85_left_finger_link" />
-            <origin xyz="0.03152616 0.0 -0.00376347" rpy="0 0 0" />
-        </joint>
-        <joint name="${prefix}robotiq_85_right_finger_joint" type="fixed">
-            <parent link="${prefix}robotiq_85_right_knuckle_link" />
-            <child link="${prefix}robotiq_85_right_finger_link" />
-            <origin xyz="-0.03152616 0.0 -0.00376347" rpy="0 0 0" />
-        </joint>
-        <joint name="${prefix}robotiq_85_left_inner_knuckle_joint" type="revolute">
-            <parent link="${prefix}robotiq_85_base_link" />
-            <child link="${prefix}robotiq_85_left_inner_knuckle_link" />
-            <axis xyz="0 -1 0" />
-            <origin xyz="0.0127 0.0 0.06142" rpy="0 0 0" />
-            <dynamics damping="0.5" friction="0.1"/>
-            <limit lower="0.0" upper="0.8" velocity="0.5" effort="50" />
-        </joint>
-        <joint name="${prefix}robotiq_85_right_inner_knuckle_joint" type="revolute">
-            <parent link="${prefix}robotiq_85_base_link" />
-            <child link="${prefix}robotiq_85_right_inner_knuckle_link" />
-            <axis xyz="0 -1 0" />
-            <origin xyz="-0.0127 0.0 0.06142" rpy="0 0 0" />
-            <dynamics damping="0.5" friction="0.1" />
-            <limit lower="-0.8" upper="0.0" velocity="0.5" effort="50" />
-        </joint>
-        <joint name="${prefix}robotiq_85_left_finger_tip_joint" type="revolute">
-            <parent link="${prefix}robotiq_85_left_finger_link" />
-            <child link="${prefix}robotiq_85_left_finger_tip_link" />
-            <axis xyz="0 -1 0" />
-            <origin xyz="0.00563134 0.0 0.04718515" rpy="0 0 0" />
-            <dynamic damping="0.5" friction="0.1" />
-            <limit lower="-0.8" upper="0.0" velocity="0.5" effort="50" />
-        </joint>
-        <joint name="${prefix}robotiq_85_right_finger_tip_joint" type="revolute">
-            <parent link="${prefix}robotiq_85_right_finger_link" />
-            <child link="${prefix}robotiq_85_right_finger_tip_link" />
-            <axis xyz="0 -1 0" />
-            <origin xyz="-0.00563134 0.0 0.04718515" rpy="0 0 0" />
-            <dynamics damping="0.5" friction="0.1" />
-            <limit lower="0.0" upper="0.8" velocity="0.5" effort="50" />
-        </joint>
+        <xacro:macro name="finger_instance" params="number yaw">
+            <link name="${prefix}robotiq_85_finger_${number}_knuckle_link">
+                <visual>
+                    <geometry>
+                        <mesh filename="package://robotiq_description/meshes/visual/2f_85/left_knuckle.dae" />
+                    </geometry>
+                </visual>
+                <collision>
+                    <geometry>
+                        <mesh filename="package://robotiq_description/meshes/collision/2f_85/left_knuckle.stl" />
+                    </geometry>
+                </collision>
+                <inertial>
+                    <origin xyz="0.01213197 0.0002 -0.00058647" rpy="0 0 0" />
+                    <mass value="1.384773208e-02" />
+                    <inertia ixx="3.5232e-7" iyy="2.31944e-6" izz="2.23136e-6" ixy="0.0" ixz="1.1744e-7" iyz="0" />
+                </inertial>
+            </link>
+            <link name="${prefix}robotiq_85_finger_${number}_finger_link">
+                <visual>
+                    <geometry>
+                        <mesh filename="package://robotiq_description/meshes/visual/2f_85/left_finger.dae" />
+                    </geometry>
+                </visual>
+                <collision>
+                    <geometry>
+                        <mesh filename="package://robotiq_description/meshes/collision/2f_85/left_finger.stl" />
+                    </geometry>
+                </collision>
+                <inertial>
+                    <origin xyz="0.00346899 -0.00079447 0.01867121" rpy="0 0 0" />
+                    <mass value="4.260376752e-02" />
+                    <inertia ixx="1.385792000000000e-05" iyy="1.183208e-05" izz="5.19672e-06" ixy="0.0" ixz="-2.17264e-06" iyz="0.0" />
+                </inertial>
+            </link>
+            <link name="${prefix}robotiq_85_finger_${number}_inner_knuckle_link">
+                <visual>
+                    <geometry>
+                        <mesh filename="package://robotiq_description/meshes/visual/2f_85/left_inner_knuckle.dae" />
+                    </geometry>
+                </visual>
+                <collision>
+                    <geometry>
+                        <mesh filename="package://robotiq_description/meshes/collision/2f_85/left_inner_knuckle.stl" />
+                    </geometry>
+                </collision>
+                <inertial>
+                    <origin xyz="0.01897699 0.00015001 0.02247101" rpy="0 0 0" />
+                    <mass value="2.969376448e-02" />
+                    <inertia ixx="9.57136e-06" iyy="8.69056e-06" izz="8.19144e-06" ixy="0.0" ixz="-3.93424e-06" iyz="0.0" />
+                </inertial>
+            </link>
+            <link name="${prefix}robotiq_85_finger_${number}_finger_tip_link">
+                <visual>
+                    <geometry>
+                        <mesh filename="package://robotiq_description/meshes/visual/2f_85/left_finger_tip.dae" />
+                    </geometry>
+                </visual>
+                <collision>
+                    <geometry>
+                        <mesh filename="package://robotiq_description/meshes/collision/2f_85/left_finger_tip.stl" />
+                    </geometry>
+                    <surface>
+                        <friction>
+                        <ode>
+                            <mu1>100000.0</mu1>
+                            <mu2>100000.0</mu2>
+                        </ode>
+                        </friction>
+                        <contact>
+                        <ode>
+                            <kp>1e+5</kp>
+                            <kd>1</kd>
+                            <soft_cfm>0</soft_cfm>
+                            <soft_erp>0.2</soft_erp>
+                            <minDepth>0.002</minDepth>
+                            <maxVel>0</maxVel>
+                        </ode>
+                        </contact>
+                    </surface>
+                </collision>
+                <inertial>
+                    <origin xyz="-0.01456706 -0.0008 0.01649701" rpy="0 0 0" />
+                    <mass value="4.268588744e-02" />
+                    <inertia ixx="1.048152e-05" iyy="1.197888e-05" izz="4.22784e-06" ixy="0.0" ixz="3.5232e-6" iyz="0.0" />
+                </inertial>
+            </link>
+            <joint name="${prefix}robotiq_85_finger_${number}_knuckle_joint" type="revolute">
+                <parent link="${prefix}robotiq_85_base_link" />
+                <child link="${prefix}robotiq_85_finger_${number}_knuckle_link" />
+                <axis xyz="0 -1 0" />
+                <origin xyz="${0.03060114 * cos(yaw)} ${0.03060114 * sin(yaw)} 0.05490452" rpy="0 0 ${yaw}" />
+                <limit lower="0.0" upper="0.8" velocity="0.5" effort="50" />
+            </joint>
+            <joint name="${prefix}robotiq_85_finger_${number}_finger_joint" type="fixed">
+                <parent link="${prefix}robotiq_85_finger_${number}_knuckle_link" />
+                <child link="${prefix}robotiq_85_finger_${number}_finger_link" />
+                <origin xyz="0.03152616 0.0 -0.00376347" rpy="0 0 0" />
+            </joint>
+            <joint name="${prefix}robotiq_85_finger_${number}_inner_knuckle_joint" type="revolute">
+                <parent link="${prefix}robotiq_85_base_link" />
+                <child link="${prefix}robotiq_85_finger_${number}_inner_knuckle_link" />
+                <axis xyz="0 -1 0" />
+                <origin xyz="${0.0127 * cos(yaw)} ${0.0127 * sin(yaw)} 0.06142" rpy="0 0 ${yaw}" />
+                <dynamics damping="0.5" friction="0.1"/>
+                <limit lower="0.0" upper="0.8" velocity="0.5" effort="50" />
+            </joint>
+            <joint name="${prefix}robotiq_85_finger_${number}_finger_tip_joint" type="revolute">
+                <parent link="${prefix}robotiq_85_finger_${number}_finger_link" />
+                <child link="${prefix}robotiq_85_finger_${number}_finger_tip_link" />
+                <axis xyz="0 -1 0" />
+                <origin xyz="0.00563134 0.0 0.04718515" rpy="0 0 0" />
+                <dynamics damping="0.5" friction="0.1" />
+                <limit lower="-0.8" upper="0.0" velocity="0.5" effort="50" />
+            </joint>
+        </xacro:macro>
+        <xacro:finger_instance number="1" yaw="0.0" />
+        <xacro:finger_instance number="2" yaw="${2.0 * pi / 3.0}" />
+        <xacro:finger_instance number="3" yaw="${4.0 * pi / 3.0}" />
     </xacro:macro>
 </robot>
